Commit message: Add files via upload
tracks added and camera removed

File: alphabot2_world/robots/alphabot2.xacro (robot description, xacro)
@@ -50,5 +50,5 @@
   <!-- end of joint for left wheel -->
   <!-- Lower Camera-->
-  <link name="lower_camera_link">
+<!--  <link name="lower_camera_link">
     <inertial>
       <mass value="0.0225"/>
@@ -70,5 +70,5 @@
     </visual>
   </link>
-  <joint name="joint_lower_camera_link" type="continuous"><!--AQUI USAM REVOLUTE -->
+  <joint name="joint_lower_camera_link" type="continuous">
     <origin rpy="0 0 0" xyz="0 0 0.045"/>
     <child link="lower_camera_link" />
@@ -80,6 +80,6 @@
   <gazebo reference="lower_camera_link">
         <material>Gazebo/Yellow</material>
-        <!--selfCollide>false</selfCollide>
-        <turnGravityOff>true</turnGravityOff-->
+ (estava comentado)     <  selfCollide>false</selfCollide>
+        <turnGravityOff>true</turnGravityOff> (fim comentado)
   </gazebo>
   <transmission name="pan_trans">
@@ -91,8 +91,8 @@
       <mechanicalReduction>1</mechanicalReduction>
     </actuator>
-  </transmission>
+  </transmission> -->
   <!--End Lower Camera-->
   <!--Upper Camera-->
-  <link name="upper_camera_link">
+ <!-- <link name="upper_camera_link">
     <origin rpy="0 0 0" xyz="0 0 0"/>
     <inertial>
@@ -117,9 +117,9 @@
   <gazebo reference="upper_camera_link">
         <material>Gazebo/Yellow</material>
-        <!--selfCollide>true</selfCollide>
-        <turnGravityOff>true</turnGravityOff-->
+        < (estava comentado) selfCollide>true</selfCollide>
+        <turnGravityOff>true</turnGravityOff  (fim comentado)>
   </gazebo>
   <joint name="joint_upper_camera_link" type="revolute">
-    <origin rpy="0 0 0" xyz="0 0 0.045"/> <!--0.045-->
+    <origin rpy="0 0 0" xyz="0 0 0.045"/>
     <child link="upper_camera_link" />
     <parent link="lower_camera_link"/>
@@ -136,5 +136,5 @@
       <mechanicalReduction>1</mechanicalReduction>
     </actuator>
-  </transmission>
+  </transmission> -->
   <!--End Upper Camera-->
   <!--For all the transmission tags; links gazebo with ROS-->
@@ -145,5 +145,5 @@
   </gazebo>
   <!-- camera -->
-  <gazebo reference="upper_camera_link">
+ <!-- <gazebo reference="upper_camera_link">
     <sensor name="alphabot2_camera" type="camera" >
       <visualize>1</visualize>
@@ -167,7 +167,4 @@
         <noise>
           <type>gaussian</type>
-          <!-- Noise is sampled independently per pixel on each frame.
-               That pixel's noise value is added to each of its color
-               channels, which at that point lie in the range [0,1]. -->
           <mean>0.0</mean>
           <stddev>0.007</stddev>
@@ -189,5 +186,5 @@
       </plugin>
     </sensor>
-  </gazebo>
+  </gazebo> -->
   <joint name="sensor1_joint" type="fixed">
     <axis xyz="0 1 0" />
